Commit message: Hardware demo (#6)

File: urdf/ur5_on_table_joint_limited.urdf.xacro (robot description, xacro)
@@ -9,5 +9,11 @@
   <!-- arm joint limited -->
   <xacro:arg name="kinematics_config" default="$(find ur_description)/config/ur5_default.yaml"/>
-  <xacro:ur5_robot prefix="" joint_limited="false"
+  <xacro:ur5_robot prefix="" joint_limited="true"
+    shoulder_pan_lower_limit="${-pi}" shoulder_pan_upper_limit="${pi}"
+    shoulder_lift_lower_limit="${-pi}" shoulder_lift_upper_limit="${pi}"
+    elbow_joint_lower_limit="${-pi}" elbow_joint_upper_limit="${pi}"
+    wrist_1_lower_limit="${-pi}" wrist_1_upper_limit="${pi}"
+    wrist_2_lower_limit="${-pi}" wrist_2_upper_limit="${pi}"
+    wrist_3_lower_limit="${-pi}" wrist_3_upper_limit="${pi}"
     transmission_hw_interface="$(arg transmission_hw_interface)"
     kinematics_file="${load_yaml('$(arg kinematics_config)')}"/>

File: urdf/ur5_robot.urdf.xacro (robot description, xacro)
@@ -7,27 +7,15 @@
   <!-- ur5 -->
   <xacro:include filename="$(find ur_description)/urdf/ur5.urdf.xacro" />
-  <!-- arm joint limited -->
+  <!-- arm -->
   <xacro:arg name="kinematics_config" default="$(find ur_description)/config/ur5_default.yaml"/>
   <xacro:ur5_robot prefix="" joint_limited="false"
     transmission_hw_interface="$(arg transmission_hw_interface)"
-    kinematics_file="${load_yaml('$(arg kinematics_config)')}"/>
-  <link name="table">
-    <visual>
-      <geometry>
-        <box size="1.25 1.25 0.25"/>
-      </geometry>
-        <origin rpy="0 0 0.0" xyz="0.0 0 -0.125"/>
-    </visual>
-  </link>
-  <joint name="table_joint" type="fixed">
-    <parent link="table" />
+    kinematics_file="${load_yaml('$(arg kinematics_config)')}"
+  />
+  <link name="world" />
+  <joint name="world_joint" type="fixed">
+    <parent link="world" />
     <child link = "base_link" />
     <origin xyz="0.0 0.0 0.0" rpy="0.0 0.0 0.0" />
   </joint>
-  <link name="world" />
-  <joint name="world_joint" type="fixed">
-    <parent link="world" />
-    <child link = "table" />
-    <origin xyz="0.0 0.0 0.0" rpy="0.0 0.0 0.0" />
-  </joint>
 </robot>
