Commit message: enable robotiq rather than stand in

File: urdf/ur5_on_table.urdf.xacro (robot description, xacro)
@@ -20,9 +20,9 @@
     <!-- transmission_hw_interface="$(arg transmission_hw_interface)"/> -->
   <!-- Robotiq -->
-  <!-- <xacro:include filename="$(find robotiq_2f_model)/model/robotiq_2f_85.urdf.xacro" /> -->
-  <!-- <xacro:robotiq_2f_85  name="robotiq_2f_85" parent="tool0"> -->
-    <!-- <origin xyz="0.0 0.0 0.0" rpy="0.0 0.0 0.0" /> -->
-  <!-- </xacro:robotiq_2f_85> -->
-  <link name="tool_link">
+  <xacro:include filename="$(find robotiq_2f_model)/model/robotiq_2f_85.urdf.xacro" />
+  <xacro:robotiq_2f_85  name="robotiq_2f_85" parent="tool0">
+    <origin xyz="0.0 0.0 0.0" rpy="0.0 0.0 0.0" />
+  </xacro:robotiq_2f_85>
+<!--   <link name="tool_link">
     <visual>
       <origin xyz="0 0 0.125"/>
@@ -39,5 +39,5 @@
     <child link="tool_link"/>
     <origin rpy="0 0 0" xyz="0 0 0"/>
-  </joint>
+  </joint> -->
   <link name="table">
     <visual>

Commit message: minor fixup to robotiq

File: urdf/ur5_on_table.urdf.xacro (robot description, xacro)
@@ -40,4 +40,11 @@
     <origin rpy="0 0 0" xyz="0 0 0"/>
   </joint> -->
+  <!-- tool center point -->
+  <link name="tool_center_point" />
+  <joint name="tool_center_point_joint" type="fixed">
+    <parent link="tool0"/>
+    <child link = "tool_center_point" />
+    <origin xyz="0.0 0.0 0.125" rpy="0.0 -1.5707 0.0" />
+  </joint>
   <link name="table">
     <visual>

Commit message: prep for hardware demo

File: urdf/ur5_on_table.urdf.xacro (robot description, xacro)
@@ -26,7 +26,7 @@
   <link name="tool_link">
     <visual>
-      <origin xyz="0 0 0.125"/>
+      <origin xyz="0 0 0.025"/>
       <geometry>
-        <cylinder length="0.25" radius="0.06"/>
+        <cylinder length="0.05" radius="0.06"/>
       </geometry>
       <material name="green">

Commit message: beta driver working

File: urdf/ur5_on_table.urdf.xacro (robot description, xacro)
@@ -25,4 +25,10 @@
     <origin xyz="0.0 0.0 0.0" rpy="0.0 0.0 0.0" />
   </joint>
+  <link name="world" />
+  <joint name="world_joint" type="fixed">
+    <parent link="world" />
+    <child link = "table" />
+    <origin xyz="0.0 0.0 0.0" rpy="0.0 0.0 0.0" />
+  </joint>
   <!-- Robotiq -->
   <!-- <xacro:include filename="$(find robotiq_2f_model)/model/robotiq_2f_85.urdf.xacro" /> -->

File: urdf/ur5_on_table_joint_limited.urdf.xacro (robot description, xacro)
@@ -31,4 +31,10 @@
     <origin xyz="0.0 0.0 0.0" rpy="0.0 0.0 0.0" />
   </joint>
+  <link name="world" />
+  <joint name="world_joint" type="fixed">
+    <parent link="world" />
+    <child link = "table" />
+    <origin xyz="0.0 0.0 0.0" rpy="0.0 0.0 0.0" />
+  </joint>
   <!-- Robotiq -->
   <!-- <xacro:include filename="$(find robotiq_2f_model)/model/robotiq_2f_85.urdf.xacro" /> -->

Commit message: removing commented out code

File: urdf/ur5_on_table.urdf.xacro (robot description, xacro)
@@ -31,24 +31,3 @@
     <origin xyz="0.0 0.0 0.0" rpy="0.0 0.0 0.0" />
   </joint>
-  <!-- Robotiq -->
-  <!-- <xacro:include filename="$(find robotiq_2f_model)/model/robotiq_2f_85.urdf.xacro" /> -->
-  <!-- <xacro:robotiq_2f_85  name="robotiq_2f_85" parent="tool0"> -->
-    <!-- <origin xyz="0.0 0.0 0.0" rpy="0.0 0.0 0.0" /> -->
-  <!-- </xacro:robotiq_2f_85> -->
-  <!-- <link name="tool_link"> -->
-    <!-- <visual> -->
-      <!-- <origin xyz="0 0 0.025"/> -->
-      <!-- <geometry> -->
-        <!-- <cylinder length="0.05" radius="0.06"/> -->
-      <!-- </geometry> -->
-      <!-- <material name="green"> -->
-        <!-- <color rgba="0 1 0 1"/> -->
-      <!-- </material> -->
-    <!-- </visual> -->
-  <!-- </link> -->
-  <!-- <joint name="$tool_link_joint" type="fixed"> -->
-    <!-- <parent link="tool0"/> -->
-    <!-- <child link="tool_link"/> -->
-    <!-- <origin rpy="0 0 0" xyz="0 0 0"/> -->
-  <!-- </joint> -->
 </robot>

File: urdf/ur5_on_table_joint_limited.urdf.xacro (robot description, xacro)
@@ -37,24 +37,3 @@
     <origin xyz="0.0 0.0 0.0" rpy="0.0 0.0 0.0" />
   </joint>
-  <!-- Robotiq -->
-  <!-- <xacro:include filename="$(find robotiq_2f_model)/model/robotiq_2f_85.urdf.xacro" /> -->
-  <!-- <xacro:robotiq_2f_85  name="robotiq_2f_85" parent="tool0"> -->
-    <!-- <origin xyz="0.0 0.0 0.0" rpy="0.0 0.0 0.0" /> -->
-  <!-- </xacro:robotiq_2f_85> -->
-  <!-- <link name="tool_link"> -->
-    <!-- <visual> -->
-      <!-- <origin xyz="0 0 0.025"/> -->
-      <!-- <geometry> -->
-        <!-- <cylinder length="0.05" radius="0.06"/> -->
-      <!-- </geometry> -->
-      <!-- <material name="green"> -->
-        <!-- <color rgba="0 1 0 1"/> -->
-      <!-- </material> -->
-    <!-- </visual> -->
-  <!-- </link> -->
-  <!-- <joint name="$tool_link_joint" type="fixed"> -->
-    <!-- <parent link="tool0"/> -->
-    <!-- <child link="tool_link"/> -->
-    <!-- <origin rpy="0 0 0" xyz="0 0 0"/> -->
-  <!-- </joint> -->
 </robot>

Commit message: config for robotiq gripper used in deep grasp
The robotiq 85 gripper is included in the collision matrix and the
driver is launched when fake_execution:=false.

File: urdf/ur5_on_table.urdf.xacro (robot description, xacro)
@@ -12,5 +12,5 @@
     transmission_hw_interface="$(arg transmission_hw_interface)"
     kinematics_file="${load_yaml('$(arg kinematics_config)')}"/>
-  <link name="table">
+  <!-- <link name="table">
     <visual>
       <geometry>
@@ -19,4 +19,9 @@
         <origin rpy="0 0 0.0" xyz="0.0 0 -0.125"/>
     </visual>
+    <collision>
+      <geometry>
+        <box size="1.25 1.25 0.25"/>
+      </geometry>
+    </collision>
   </link>
   <joint name="table_joint" type="fixed">
@@ -30,4 +35,10 @@
     <child link = "table" />
     <origin xyz="0.0 0.0 0.0" rpy="0.0 0.0 0.0" />
+  </joint> -->
+  <link name="world" />
+  <joint name="world_joint" type="fixed">
+    <parent link="world" />
+    <child link = "base_link" />
+    <origin xyz="0.0 0.0 0.0" rpy="0.0 0.0 0.0" />
   </joint>
 </robot>

File: urdf/ur5_on_table_joint_limited.urdf.xacro (robot description, xacro)
@@ -18,5 +18,11 @@
     transmission_hw_interface="$(arg transmission_hw_interface)"
     kinematics_file="${load_yaml('$(arg kinematics_config)')}"/>
-  <link name="table">
+  <link name="world" />
+  <joint name="world_joint" type="fixed">
+    <parent link="world" />
+    <child link = "base_link" />
+    <origin xyz="0.0 0.0 0.0" rpy="0.0 0.0 0.0" />
+  </joint>
+  <!-- <link name="table">
     <visual>
       <geometry>
@@ -25,4 +31,9 @@
         <origin rpy="0 0 0.0" xyz="0.0 0 -0.125"/>
     </visual>
+    <collision>
+      <geometry>
+        <box size="1.25 1.25 0.25"/>
+      </geometry>
+    </collision>
   </link>
   <joint name="table_joint" type="fixed">
@@ -36,4 +47,12 @@
     <child link = "table" />
     <origin xyz="0.0 0.0 0.0" rpy="0.0 0.0 0.0" />
-  </joint>
+  </joint> -->
+  <!-- Tool changer -->
+    <xacro:include filename="$(find robotiq_85_description)/urdf/tool_changer.xacro" />
+    <xacro:tool_changer prefix="" connected_to="tool0"/>
+  <!-- GRIPPER -->
+  <xacro:include filename="$(find robotiq_85_description)/urdf/robotiq_85_gripper.urdf.xacro" />
+  <xacro:robotiq_85_gripper prefix="" parent="tool_changer_tool0" >
+        <origin xyz="0.0 0.0 0.0" rpy="0.0 -1.57 0.0"/>
+  </xacro:robotiq_85_gripper>
 </robot>
