Commit message: Add Hokoyu to UR5 - Part 1

File: urdf/ur5_3Dsensor.urdf.xacro (robot description, xacro)
@@ -14,22 +14,34 @@
   <xacro:ur5_robot prefix="" joint_limited="false"
     transmission_hw_interface="$(arg transmission_hw_interface)"/>
-  <link name="table">
-    <visual>
+  <link name="hokuyo">
+    <visual name='hokuyo_visual'>
+      <origin xyz="0 0 0" rpy=" 0 0 0"/>
       <geometry>
-        <box size="1.25 1.25 0.25"/>
+        <mesh filename="$(find picknik_ur5_moveit_config)/meshes/hokuyo.dae"/>
       </geometry>
-        <origin rpy="0 0 0.0" xyz="0.0 0 -0.125"/>
     </visual>
+    <inertial>
+      <mass value="1e-5"/>
+      <origin xyz="0 0 0" rpy=" 0 0 0"/>
+      <inertia
+          ixx="1e-6" ixy="0" ixz="0"
+          iyy="1e-6" iyz="0"
+          izz="1e-6"
+      />
+    </inertial>
+    <collision name='camera_collision'>
+      <origin xyz="0 0 0" rpy=" 0 0 0"/>
+      <geometry>
+        <box size=".1 .1 .1"/>
+      </geometry>
+    </collision>
   </link>
-  <joint name="table_joint" type="fixed">
-    <parent link="table" />
-    <child link = "base_link" />
-    <origin xyz="0.0 0.0 0.0" rpy="0.0 0.0 0.0" />
-  </joint>
-  <link name="world" />
-  <joint name="world_joint" type="fixed">
-    <parent link="world" />
-    <child link = "table" />
-    <origin xyz="0.0 0.0 0.0" rpy="0.0 0.0 0.0" />
+  <joint type="fixed" name="hokuyo_joint">
+    <origin xyz="0.15 0 0.1" rpy="0 0 0"/>
+    <child link="hokuyo"/>
+    <parent link="base_link"/>
+    <axis xyz="0 1 0" rpy="0 0 0"/>
+    <limit effort="10000" velocity="1000"/>
+    <dynamics damping="1.0" friction="1.0"/>
   </joint>
 </robot>

Commit message: Added hokoyu to table - Need to fix physics

File: urdf/ur5_3Dsensor.urdf.xacro (robot description, xacro)
@@ -5,4 +5,5 @@
   <!-- common stuff -->
   <xacro:include filename="$(find ur_description)/urdf/common.gazebo.xacro" />
+  <include filename="$(find picknik_ur5_moveit_config)/urdf/ur5_sensor.gazebo" />
   <!-- ur5 -->
   <xacro:include filename="$(find ur_description)/urdf/ur5.urdf.xacro" />
@@ -38,10 +39,23 @@
   </link>
   <joint type="fixed" name="hokuyo_joint">
-    <origin xyz="0.15 0 0.1" rpy="0 0 0"/>
+    <origin xyz="0.15 -1 0.1" rpy="0 0 0"/>
     <child link="hokuyo"/>
-    <parent link="base_link"/>
+    <parent link="table"/>
     <axis xyz="0 1 0" rpy="0 0 0"/>
     <limit effort="10000" velocity="1000"/>
     <dynamics damping="1.0" friction="1.0"/>
   </joint>
+  <link name="table">
+    <visual>
+      <origin rpy="0 0 0" xyz="0 -0.45 -0.03"/>
+      <geometry>
+        <box size="0.6 1.2 0.05"/>
+      </geometry>
+      <material name="grey"/>
+    </visual>
+  </link>
+  <joint name="table_joint" type="fixed">
+    <parent link="table"/>
+    <child link="base_link"/>
+  </joint>
 </robot>

Commit message: Add kinect support

File: urdf/ur5_3Dsensor.urdf.xacro (robot description, xacro)
@@ -17,7 +17,7 @@
   <link name="hokuyo">
     <visual name='hokuyo_visual'>
-      <origin xyz="0 0 0" rpy=" 0 0 0"/>
+      <origin xyz="0 0 0" rpy="0 0 0"/>
       <geometry>
-        <mesh filename="$(find picknik_ur5_moveit_config)/meshes/hokuyo.dae"/>
+        <mesh filename="$(find picknik_ur5_moveit_config)/kinect/meshes/kinect.dae"/>
       </geometry>
     </visual>
@@ -46,4 +46,13 @@
     <dynamics damping="1.0" friction="1.0"/>
   </joint>
+  <joint type="fixed" name="sensor_joint">
+    <origin xyz="0 0 0" rpy="1.57 0 1.57"/>
+    <child link="sensor"/>
+    <parent link="hokuyo"/>
+    <axis xyz="1 0 0" rpy="0 0 0"/>
+    <limit effort="10000" velocity="1000"/>
+    <dynamics damping="1.0" friction="1.0"/>
+  </joint>
+  <link name="sensor"/>
   <link name="table">
     <visual>

Commit message: Working version

File: urdf/ur5_3Dsensor.urdf.xacro (robot description, xacro)
@@ -46,13 +46,4 @@
     <dynamics damping="1.0" friction="1.0"/>
   </joint>
-  <joint type="fixed" name="sensor_joint">
-    <origin xyz="0 0 0" rpy="1.57 0 1.57"/>
-    <child link="sensor"/>
-    <parent link="hokuyo"/>
-    <axis xyz="1 0 0" rpy="0 0 0"/>
-    <limit effort="10000" velocity="1000"/>
-    <dynamics damping="1.0" friction="1.0"/>
-  </joint>
-  <link name="sensor"/>
   <link name="table">
     <visual>
@@ -63,4 +54,10 @@
       <material name="grey"/>
     </visual>
+    <collision name='camera_collision'>
+      <origin rpy="0 0 0" xyz="0 -0.45 -0.03"/>
+      <geometry>
+        <box size="0.6 1.2 0.05"/>
+      </geometry>
+    </collision>
   </link>
   <joint name="table_joint" type="fixed">
@@ -68,3 +65,78 @@
     <child link="base_link"/>
   </joint>
+   <joint name="camera_rgb_joint" type="fixed">
+    <origin rpy="0 0 1.57" xyz="0 0 0"/>
+    <parent link="hokuyo"/>
+    <child link="camera_rgb_frame"/>
+  </joint>
+  <link name="camera_rgb_frame">
+    <inertial>
+      <mass value="0.001"/>
+      <origin xyz="0 0 0"/>
+      <inertia ixx="0.0001" ixy="0.0" ixz="0.0" iyy="0.0001" iyz="0.0" izz="0.0001"/>
+    </inertial>
+  </link>
+  <joint name="camera_rgb_optical_joint" type="fixed">
+    <origin rpy="-1.57079632679 0 -1.57079632679" xyz="0 0 0"/>
+    <parent link="camera_rgb_frame"/>
+    <child link="camera_rgb_optical_frame"/>
+  </joint>
+  <link name="camera_rgb_optical_frame">
+    <inertial>
+      <mass value="0.001"/>
+      <origin xyz="0 0 0"/>
+      <inertia ixx="0.0001" ixy="0.0" ixz="0.0" iyy="0.0001" iyz="0.0" izz="0.0001"/>
+    </inertial>
+  </link>
+  <joint name="camera_joint" type="fixed">
+    <origin rpy="0 0 0" xyz="-0.031 -0.0 -0.016"/>
+    <parent link="camera_rgb_frame"/>
+    <child link="camera_link"/>
+  </joint>
+  <link name="camera_link">
+    <visual>
+      <origin rpy="0 0 1.57079632679" xyz="0 0 0"/>
+      <geometry>
+        <mesh filename="package://picknik_ur5_moveit_config/kinect/meshes/kinect.dae"/>
+      </geometry>
+    </visual>
+    <collision>
+      <origin rpy="0 0 0" xyz="0.0 0.0 0.0"/>
+      <geometry>
+        <box size="0.07271 0.27794 0.073"/>
+      </geometry>
+    </collision>
+    <inertial>
+      <mass value="0.001"/>
+      <origin xyz="0 0 0"/>
+      <inertia ixx="0.0001" ixy="0.0" ixz="0.0" iyy="0.0001" iyz="0.0" izz="0.0001"/>
+    </inertial>
+  </link>
+  <!-- The fixed joints & links below are usually published by static_transformers launched by the OpenNi launch
+     files. However, for Gazebo simulation we need them, so we add them here.
+     (Hence, don't publish them additionally!) -->
+  <joint name="camera_depth_joint" type="fixed">
+    <origin rpy="0 0 0" xyz="0 0.0 0"/>
+    <parent link="camera_rgb_frame"/>
+    <child link="camera_depth_frame"/>
+  </joint>
+  <link name="camera_depth_frame">
+    <inertial>
+      <mass value="0.001"/>
+      <origin xyz="0 0 0"/>
+      <inertia ixx="0.0001" ixy="0.0" ixz="0.0" iyy="0.0001" iyz="0.0" izz="0.0001"/>
+    </inertial>
+  </link>
+  <joint name="camera_depth_optical_joint" type="fixed">
+    <origin rpy="-1.57079632679 0 -1.57079632679" xyz="0 0 0"/>
+    <parent link="camera_depth_frame"/>
+    <child link="camera_depth_optical_frame"/>
+  </joint>
+  <link name="camera_depth_optical_frame">
+    <inertial>
+      <mass value="0.001"/>
+      <origin xyz="0 0 0"/>
+      <inertia ixx="0.0001" ixy="0.0" ixz="0.0" iyy="0.0001" iyz="0.0" izz="0.0001"/>
+    </inertial>
+  </link>
 </robot>

Commit message: Mesh Filter launch file

File: urdf/ur5_3Dsensor.urdf.xacro (robot description, xacro)
@@ -8,12 +8,7 @@
   <!-- ur5 -->
   <xacro:include filename="$(find ur_description)/urdf/ur5.urdf.xacro" />
-  <!-- arm joint limited -->
-  <!-- <xacro:arg name="kinematics_config" default="$(find ur_description)/config/ur5_default.yaml"/>
-  <xacro:ur5_robot prefix="" joint_limited="false"
-    transmission_hw_interface="$(arg transmission_hw_interface)"
-    kinematics_file="${load_yaml('$(arg kinematics_config)')}"/> -->
   <xacro:ur5_robot prefix="" joint_limited="false"
     transmission_hw_interface="$(arg transmission_hw_interface)"/>
-  <link name="hokuyo">
+  <link name="kinect">
     <visual name='hokuyo_visual'>
       <origin xyz="0 0 0" rpy="0 0 0"/>
@@ -40,5 +35,5 @@
   <joint type="fixed" name="hokuyo_joint">
     <origin xyz="0.15 -1 0.1" rpy="0 0 0"/>
-    <child link="hokuyo"/>
+    <child link="kinect"/>
     <parent link="table"/>
     <axis xyz="0 1 0" rpy="0 0 0"/>
@@ -67,5 +62,5 @@
    <joint name="camera_rgb_joint" type="fixed">
     <origin rpy="0 0 1.57" xyz="0 0 0"/>
-    <parent link="hokuyo"/>
+    <parent link="kinect"/>
     <child link="camera_rgb_frame"/>
   </joint>
